Commit message: modified mutiple launch files

File: joined_scout_ur5e/urdf/scout_UR5e.xacro (robot description, xacro)
@@ -3,5 +3,5 @@
   xmlns:xacro="http://wiki.ros.org/xacro">
     <!-- include xacro file containing a link where you want to attach the manipulator -->
-    <xacro:include filename="$(find joined_scout_ur5e)/urdf/scout_v2.xacro"/>
+    <xacro:include filename="$(find scout_description)/urdf/scout_v2.xacro"/>
     <xacro:include filename="$(find ur_e_description)/urdf/common.gazebo.xacro" />
     <!-- ur5e -->
@@ -9,35 +9,11 @@
     <!-- arm -->
     <xacro:arg name="kinematics_config" default="$(find ur_e_description)/config/ur5e_default.yaml"/>
-    <xacro:ur5e_robot prefix="" joint_limited="true"
+    <xacro:ur5e_robot prefix="ur_" joint_limited="true"
     kinematics_file="${load_yaml('$(arg kinematics_config)')}"
     />
-    <link name="dual_world"/>
-    <link name="dual_base_link"/>
-    <joint name="dual_world" type="fixed">
-        <parent link="dual_world"/>
-        <child link="dual_base_link"/>
-        <origin xyz="0 0 0" rpy="0 0 0" />
-    </joint>
-    <link name="ur_world" />
-    <joint name="ur_world_joint" type="fixed">
-        <parent link="ur_world" />
-        <child link = "base_link" />
-        <origin xyz="0.0 0.0 0.0" rpy="0.0 0.0 0.0" />
-    </joint>
-    <link name="scout_world"/>
-    <joint name="scout_world_joint" type="fixed">
-        <parent link="scout_world" />
-        <child link = "scout_base_link" />  <!--"r_base_link" is follow the prefix setting.-->
-        <origin xyz="0 0 0" rpy="0 0 0" />
-    </joint>
-    <joint name="ur_joint" type="fixed">
-        <parent link="dual_base_link"/>
-        <child link="ur_world"/>
-        <origin xyz="0 0 0.13" rpy="0 0 0" />
-    </joint>
-    <joint name="scout_joint" type="fixed">
-        <parent link="dual_base_link"/>
-        <child link="scout_world"/>
-        <origin xyz="0 0 0" rpy="0 0 0" />
+    <joint name="dual_joint" type="fixed">
+        <parent link="base_link"/>
+        <child link="ur_base_link"/>
+        <origin xyz="0 0 0.20" rpy="0 0 0" />
     </joint>
 </robot>

File: joined_scout_ur5e/urdf/scout_v2.xacro (robot description, xacro)
@@ -14,9 +14,9 @@
     <xacro:property name="wheelbase" value="0.498" />
     <xacro:property name="track" value="0.58306" />
-    <xacro:property name="wheel_vertical_offset" value="-0.2002" />
+    <xacro:property name="wheel_vertical_offset" value="-0.0702" />
     <xacro:property name="wheel_length" value="1.1653e-01" />
     <xacro:property name="wheel_radius" value="1.6459e-01" />
     <!-- Base link -->
-    <link name="scout_base_link">
+    <link name="base_link">
         <visual>
             <origin xyz="0 0 0" rpy="0 0 0" />
@@ -55,5 +55,5 @@
     <joint name="inertial_joint" type="fixed">
         <origin xyz="0 0 0" rpy="0 0 0" />
-        <parent link="scout_base_link" />
+        <parent link="base_link" />
         <child link="inertial_link" />
     </joint>

Commit message: operating

File: joined_scout_ur5e/urdf/scout_UR5e.xacro (robot description, xacro)
@@ -3,17 +3,17 @@
   xmlns:xacro="http://wiki.ros.org/xacro">
     <!-- include xacro file containing a link where you want to attach the manipulator -->
-    <xacro:include filename="$(find scout_description)/urdf/scout_v2.xacro"/>
-    <xacro:include filename="$(find ur_e_description)/urdf/common.gazebo.xacro" />
+    <xacro:include filename="$(find joined_scout_ur5e)/urdf/scout_v2.xacro"/>
+    <!-- <xacro:include filename="$(find ur_e_description)/urdf/common.gazebo.xacro" /> -->
     <!-- ur5e -->
     <xacro:include filename="$(find ur_e_description)/urdf/ur5e.urdf.xacro" />
     <!-- arm -->
     <xacro:arg name="kinematics_config" default="$(find ur_e_description)/config/ur5e_default.yaml"/>
-    <xacro:ur5e_robot prefix="ur_" joint_limited="true"
+    <xacro:ur5e_robot prefix="" joint_limited="true"
     kinematics_file="${load_yaml('$(arg kinematics_config)')}"
     />
-    <joint name="dual_joint" type="fixed">
-        <parent link="base_link"/>
-        <child link="ur_base_link"/>
-        <origin xyz="0 0 0.20" rpy="0 0 0" />
+    <joint name="joined_joint" type="fixed">
+        <parent link="scout_base_link"/>
+        <child link="base_link"/>
+        <origin xyz="0 0 0.13" rpy="0 0 0" />
     </joint>
 </robot>

File: joined_scout_ur5e/urdf/scout_v2.xacro (robot description, xacro)
@@ -4,6 +4,6 @@
     <xacro:arg name="robot_namespace" default="/" />
     <!--xacro:arg name="urdf_extras" default="empty.urdf" /-->
-    <xacro:include filename="$(find scout_description)/urdf/scout_wheel_type1.xacro" />
-    <xacro:include filename="$(find scout_description)/urdf/scout_wheel_type2.xacro" />
+    <xacro:include filename="$(find joined_scout_ur5e)/urdf/scout_wheel_type1.xacro" />
+    <xacro:include filename="$(find joined_scout_ur5e)/urdf/scout_wheel_type2.xacro" />
     <!-- Variables -->
     <xacro:property name="M_PI" value="3.14159"/>
@@ -18,5 +18,5 @@
     <xacro:property name="wheel_radius" value="1.6459e-01" />
     <!-- Base link -->
-    <link name="base_link">
+    <link name="scout_base_link">
         <visual>
             <origin xyz="0 0 0" rpy="0 0 0" />
@@ -55,5 +55,5 @@
     <joint name="inertial_joint" type="fixed">
         <origin xyz="0 0 0" rpy="0 0 0" />
-        <parent link="base_link" />
+        <parent link="scout_base_link" />
         <child link="inertial_link" />
     </joint>

Commit message: latest

File: joined_scout_ur5e/urdf/scout_UR5e.xacro (robot description, xacro)
@@ -12,4 +12,10 @@
     kinematics_file="${load_yaml('$(arg kinematics_config)')}"
     />
+    <link name="world"/>
+    <joint name="world_joint" type="fixed">
+        <parent link="world"/>
+        <child link="scout_base_link"/>
+        <origin xyz="0 0 0" rpy="0 0 0" />
+    </joint>
     <joint name="joined_joint" type="fixed">
         <parent link="scout_base_link"/>

Commit message: testing

File: joined_scout_ur5e/urdf/scout_UR5e.xacro (robot description, xacro)
@@ -6,9 +6,10 @@
     <!-- ur5e -->
     <xacro:include filename="$(find ur_e_description)/urdf/ur5e.urdf.xacro" />
+    <xacro:include filename="$(find ur_e_description)/urdf/common.gazebo.xacro" />
     <!-- arm -->
     <xacro:arg name="kinematics_config" default="$(find ur_e_description)/config/ur5e_default.yaml"/>
     <xacro:ur5e_robot prefix="" joint_limited="true" kinematics_file="${load_yaml('$(arg kinematics_config)')}"/>
     <link name="world"/>
-    <joint name="world_joint" type="fixed">
+    <joint name="world_joint" type="floating">
         <parent link="world"/>
         <child link="scout_base_link"/>

Commit message: 1/22 operable

File: joined_scout_ur5e/urdf/scout_UR5e.xacro (robot description, xacro)
@@ -6,17 +6,17 @@
     <!-- ur5e -->
     <xacro:include filename="$(find ur_e_description)/urdf/ur5e.urdf.xacro" />
-    <xacro:include filename="$(find ur_e_description)/urdf/common.gazebo.xacro" />
     <!-- arm -->
     <xacro:arg name="kinematics_config" default="$(find ur_e_description)/config/ur5e_default.yaml"/>
-    <xacro:ur5e_robot prefix="" joint_limited="true" kinematics_file="${load_yaml('$(arg kinematics_config)')}"/>
+    <xacro:arg name="prefix" default="arm_"/>
+    <xacro:ur5e_robot prefix="$(arg prefix)" joint_limited="true" kinematics_file="${load_yaml('$(arg kinematics_config)')}"/>
     <link name="world"/>
     <joint name="world_joint" type="floating">
         <parent link="world"/>
-        <child link="scout_base_link"/>
+        <child link="base_link"/>
         <origin xyz="0 0 0" rpy="0 0 0" />
     </joint>
     <joint name="joined_joint" type="fixed">
-        <parent link="scout_base_link"/>
-        <child link="base_link"/>
+        <parent link="base_link"/>
+        <child link="$(arg prefix)base_link"/>
         <origin xyz="0 0 0.13" rpy="0 0 0" />
     </joint>

File: joined_scout_ur5e/urdf/scout_v2.xacro (robot description, xacro)
@@ -2,8 +2,8 @@
 <robot name="scout_v2"
     xmlns:xacro="http://ros.org/wiki/xacro">
-    <xacro:arg name="robot_namespace" default="/" />
-    <!--xacro:arg name="urdf_extras" default="empty.urdf" /-->
-    <xacro:include filename="$(find joined_scout_ur5e)/urdf/scout_wheel_type1.xacro" />
-    <xacro:include filename="$(find joined_scout_ur5e)/urdf/scout_wheel_type2.xacro" />
+    <xacro:arg name="robot_namespace" default="" />
+    <!--xacro:arg name="urdf_extras" default="$(find scout_description)/urdf/empty.urdf" /-->
+    <xacro:include filename="$(find scout_description)/urdf/scout_wheel_type1.xacro" />
+    <xacro:include filename="$(find scout_description)/urdf/scout_wheel_type2.xacro" />
     <!-- Variables -->
     <xacro:property name="M_PI" value="3.14159"/>
@@ -18,5 +18,5 @@
     <xacro:property name="wheel_radius" value="1.6459e-01" />
     <!-- Base link -->
-    <link name="scout_base_link">
+    <link name="base_link">
         <visual>
             <origin xyz="0 0 0" rpy="0 0 0" />
@@ -45,5 +45,5 @@
     <link name="inertial_link">
         <inertial>
-            <mass value="40" />
+            <mass value="4000" />
             <!-- <mass value="50" /> -->
             <!-- <origin xyz="-0.00065 -0.085 0.062" />
@@ -55,5 +55,5 @@
     <joint name="inertial_joint" type="fixed">
         <origin xyz="0 0 0" rpy="0 0 0" />
-        <parent link="scout_base_link" />
+        <parent link="base_link" />
         <child link="inertial_link" />
     </joint>

Commit message: added 2f-85 gripper package

File: joined_scout_ur5e/urdf/scout_UR5e.xacro (robot description, xacro)
@@ -2,6 +2,7 @@
 <robot name="joinedrobot"
   xmlns:xacro="http://wiki.ros.org/xacro">
-    <!-- include xacro file containing a link where you want to attach the manipulator -->
-    <xacro:include filename="$(find joined_scout_ur5e)/urdf/scout_v2.xacro"/>
+    <xacro:arg name="robot_namespace" default="" />
+    <!-- scout 2.0 -->
+    <xacro:include filename="$(find scout_description)/urdf/scout_v2.xacro"/>
     <!-- ur5e -->
     <xacro:include filename="$(find ur_e_description)/urdf/ur5e.urdf.xacro" />
@@ -11,8 +12,14 @@
     <xacro:ur5e_robot prefix="$(arg prefix)" joint_limited="true" kinematics_file="${load_yaml('$(arg kinematics_config)')}"/>
     <link name="world"/>
-    <joint name="world_joint" type="floating">
+    <!-- <joint name="world_odom" type="fixed">
+        <parent link="world"/>
+        <child link="odom"/>
+        <origin xyz="0 0 0" rpy="0 0 0" />
+    </joint> -->
+    <joint name="world_joint" type="prismatic">
         <parent link="world"/>
         <child link="base_link"/>
         <origin xyz="0 0 0" rpy="0 0 0" />
+         <dynamics damping="0.1" friction="10.0"/>
     </joint>
     <joint name="joined_joint" type="fixed">

Commit message: fixed some arguments

File: joined_scout_ur5e/urdf/scout_UR5e.xacro (robot description, xacro)
@@ -17,9 +17,9 @@
         <origin xyz="0 0 0" rpy="0 0 0" />
     </joint> -->
-    <joint name="world_joint" type="prismatic">
+    <joint name="world_joint" type="floating">
         <parent link="world"/>
         <child link="base_link"/>
         <origin xyz="0 0 0" rpy="0 0 0" />
-         <dynamics damping="0.1" friction="10.0"/>
+        <!-- <axis xyz="0 0 1" /> -->
     </joint>
     <joint name="joined_joint" type="fixed">

Commit message: solving gazebo issue

File: joined_scout_ur5e/urdf/scout_UR5e.xacro (robot description, xacro)
@@ -2,29 +2,38 @@
 <robot name="joinedrobot"
   xmlns:xacro="http://wiki.ros.org/xacro">
-    <xacro:arg name="robot_namespace" default="" />
+    <xacro:arg name="robot_namespace" default="/" />
     <!-- scout 2.0 -->
-    <xacro:include filename="$(find scout_description)/urdf/scout_v2.xacro"/>
+    <!-- <xacro:include filename="$(find scout_description)/urdf/scout_v2.xacro"/> -->
+    <xacro:include filename="$(find joined_scout_ur5e)/urdf/scout_v2.xacro"/>
     <!-- ur5e -->
-    <xacro:include filename="$(find ur_e_description)/urdf/ur5e.urdf.xacro" />
+    <!-- <xacro:include filename="$(find ur_e_description)/urdf/ur5e.urdf.xacro" /> -->
+    <xacro:include filename="$(find joined_scout_ur5e)/urdf/ur5e.urdf.xacro" />
     <!-- arm -->
+    <xacro:include filename="$(find ur_e_description)/urdf/common.gazebo.xacro" />
     <xacro:arg name="kinematics_config" default="$(find ur_e_description)/config/ur5e_default.yaml"/>
     <xacro:arg name="prefix" default="arm_"/>
     <xacro:ur5e_robot prefix="$(arg prefix)" joint_limited="true" kinematics_file="${load_yaml('$(arg kinematics_config)')}"/>
     <link name="world"/>
-    <!-- <joint name="world_odom" type="fixed">
+    <joint name="ur_joint" type="fixed">
+        <parent link="scout_world"/>
+        <child link="ur_world"/>
+        <origin xyz="0 0 0.105" rpy="0 0 0" />
+    </joint>
+    <joint name="scout_joint" type="floating">
         <parent link="world"/>
-        <child link="odom"/>
+        <child link="scout_world"/>
         <origin xyz="0 0 0" rpy="0 0 0" />
-    </joint> -->
-    <joint name="world_joint" type="floating">
-        <parent link="world"/>
+    </joint>
+    <link name="scout_world"/>
+    <joint name="world_joint" type="fixed">
+        <parent link="scout_world"/>
         <child link="base_link"/>
         <origin xyz="0 0 0" rpy="0 0 0" />
-        <!-- <axis xyz="0 0 1" /> -->
     </joint>
+    <link name="ur_world"/>
     <joint name="joined_joint" type="fixed">
-        <parent link="base_link"/>
+        <parent link="ur_world"/>
         <child link="$(arg prefix)base_link"/>
-        <origin xyz="0 0 0.13" rpy="0 0 0" />
+        <origin xyz="0 0 0" rpy="0 0 0" />
     </joint>
 </robot>

File: joined_scout_ur5e/urdf/scout_v2.xacro (robot description, xacro)
@@ -2,5 +2,5 @@
 <robot name="scout_v2"
     xmlns:xacro="http://ros.org/wiki/xacro">
-    <xacro:arg name="robot_namespace" default="" />
+    <xacro:arg name="robot_namespace" default="/" />
     <!--xacro:arg name="urdf_extras" default="$(find scout_description)/urdf/empty.urdf" /-->
     <xacro:include filename="$(find scout_description)/urdf/scout_wheel_type1.xacro" />
@@ -45,5 +45,5 @@
     <link name="inertial_link">
         <inertial>
-            <mass value="4000" />
+            <mass value="40" />
             <!-- <mass value="50" /> -->
             <!-- <origin xyz="-0.00065 -0.085 0.062" />
